Commit message: minor bugs & more polishing

File: urdf/_d435.urdf.xacro (robot description, xacro)
@@ -8,5 +8,5 @@
 <robot name="sensor_d435" xmlns:xacro="http://ros.org/wiki/xacro">
   <!--File includes-->
-  <xacro:include filename="$(find realsense2_description)/urdf/_d435.gazebo.xacro"/>
+  <xacro:include filename="$(find sensing-aruco)/urdf/_d435.gazebo.xacro"/>
   <xacro:macro name="sensor_d435" params="name:=camera topics_ns:=camera parent *origin publish_pointcloud:=true">
     <xacro:property name="M_PI" value="3.1415926535897931" />
@@ -48,6 +48,6 @@
         <geometry>
           <!-- <box size="${d435_cam_width} ${d435_cam_height} ${d435_cam_depth}"/> -->
-          <mesh filename="package://realsense2_description/meshes/d435.dae" />
-          <!--<mesh filename="package://realsense2_description/meshes/d435/d435.dae" />-->
+          <mesh filename="package://sensing-aruco/meshes/d435.dae" />
+          <!--<mesh filename="package://sensing-aruco/meshes/d435/d435.dae" />-->
         </geometry>
         <material name="${name}_aluminum"/>

File: urdf/test_d435_camera.urdf.xacro (robot description, xacro)
@@ -1,5 +1,5 @@
 <?xml version="1.0"?>
 <robot name="realsense2_camera" xmlns:xacro="http://ros.org/wiki/xacro">
-  <xacro:include filename="$(find realsense2_description)/urdf/_d435.urdf.xacro" />
+  <xacro:include filename="$(find sensing-aruco)/urdf/_d435.urdf.xacro" />
   <link name="base_link" />
   <xacro:sensor_d435 name="camera" topics_ns="camera" parent="base_link" publish_pointcloud="true">

File: urdf/test_d435_multiple_cameras.urdf.xacro (robot description, xacro)
@@ -1,5 +1,5 @@
 <?xml version="1.0"?>
 <robot name="realsense2_camera" xmlns:xacro="http://ros.org/wiki/xacro">
-  <xacro:include filename="$(find realsense2_description)/urdf/_d435.urdf.xacro" />
+  <xacro:include filename="$(find sensing-aruco)/urdf/_d435.urdf.xacro" />
   <link name="base_link" />
   <sensor_d435 parent="base_link" name="camera1">
